File: PCB/SofleKeyboard.sch (KiCad schematic (older format))
At the start: 85 parts, among them J1 LED, J2 4PIN, J3 OLED, P1 i2c_pin, P2 i2c_pin, SW1 SW_PUSH, SW10 SW_PUSH, SW11 SW_PUSH, SW12 SW_PUSH, SW13 SW_PUSH, SW14 SW_PUSH, SW15 SW_PUSH, SW16 SW_PUSH, SW17 SW_PUSH, SW18 SW_PUSH, SW19 SW_PUSH, SW2 SW_PUSH, SW20 SW_PUSH, SW21 SW_PUSH, SW22 SW_PUSH, SW23 SW_PUSH, SW24 SW_PUSH, SW25 Rotary_Encoder_Switch, SW26 SW_PUSH, SW27 SW_PUSH, SW28 SW_PUSH, SW29 SW_PUSH, SW3 SW_PUSH, SW30 SW_PUSH, SW4 SW_PUSH, SW5 SW_PUSH, SW6 SW_PUSH, SW7 SW_PUSH, SW8 SW_PUSH, SW9 SW_PUSH, U1 ProMicro

Commit message: footprints fixed, onto layout
Parts:
- added D31, D32, D33, D34, D35, D36, D37: LED_sk2812_SM, LED_SMD:SK6812MINI_underglow_dev, symbol SofleKeyboard:LED_sk2812_SM
- added J4: key leds, Connector:3x1header, symbol SofleKeyboard-rescue:LED-Lily58-cache-Lily58_Pro-rescue
- added J5: backlight sel, Connector:3x1header, symbol SofleKeyboard-rescue:LED-Lily58-cache-Lily58_Pro-rescue
- added J6: indicator bypass, Connector:3x1header, symbol SofleKeyboard-rescue:LED-Lily58-cache-Lily58_Pro-rescue
- added unit 2 of SW1
- added unit 2 of SW10
- added unit 2 of SW11
- added unit 2 of SW12
- added unit 2 of SW13
- added unit 2 of SW14
- added unit 2 of SW15
- added unit 2 of SW16
- added unit 2 of SW17
- added unit 2 of SW18
- added unit 2 of SW19
- added unit 2 of SW2
- added unit 2 of SW20
- added unit 2 of SW21
- added unit 2 of SW22
- added unit 2 of SW23
- added unit 2 of SW24
- added unit 2 of SW26
- added unit 2 of SW27
- added unit 2 of SW28
- added unit 2 of SW29
- added unit 2 of SW3
- added unit 2 of SW30
- added unit 2 of SW4
- added unit 2 of SW5
- added unit 2 of SW6
- added unit 2 of SW7
- added unit 2 of SW8
- added unit 2 of SW9
- D1, D10, D11, D12, D13, D14, D15, D16, D17, D18, D19, D2, D20, D21, D22, D23, D24, D25, D26, D27, D28, D29, D3, D30, D4, D5, D6, D7, D8, D9: footprint SofleKeyboard-footprint:Diode_SOD123 -> Diode_SMD:crkbd-diode
- JP1, JP2, JP3, JP4, JP5, JP6, JP7, JP8: symbol Device:Jumper_NO_Small -> SofleKeyboard-rescue:Jumper_NO_Small-Device
- SW1, SW10, SW11, SW12, SW13, SW14, SW15, SW16, SW17, SW18, SW19, SW2, SW20, SW21, SW22, SW23, SW24, SW27, SW28, SW29, SW3, SW30, SW4, SW5, SW6, SW7, SW8, SW9: value SW_PUSH -> SW_PUSH-MX_W_LED; footprint SofleKeyboard-footprint:CherryMX_KailhLowProfile_Hotswap -> Button_Switch_Keyboard:SK6812MINI_and_cherry; symbol SofleKeyboard-rescue:SW_PUSH-Lily58-cache-Lily58_Pro-rescue -> SofleKeyboard:SW_PUSH-MX_W_LED
- SW25: symbol Device:Rotary_Encoder_Switch -> SofleKeyboard-rescue:Rotary_Encoder_Switch-Device
- SW26: value SW_PUSH -> SW_PUSH-MX_W_LED; footprint SofleKeyboard-footprint:CherryMX_KailhLowProfile_Hotswap_1.5 -> Button_Switch_Keyboard:SK6812MINI_and_cherry; symbol SofleKeyboard-rescue:SW_PUSH-Lily58-cache-Lily58_Pro-rescue -> SofleKeyboard:SW_PUSH-MX_W_LED
- W1: symbol Device:Jumper -> SofleKeyboard-rescue:Jumper-Device
Connections:
- net labels added: backlight, lights, underglow
- wire segments 87 -> 352
Other:
- moved on the sheet: D1, D10, D11, D12, D13, D14, D15, D16, D17, D18, D19, D2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
