File: Sofle_RGB/PCB/SofleKeyboard.sch (KiCad schematic (older format))
At the start: 95 parts, among them J1 LED, J2 4PIN, J3 OLED, J4 key leds, J5 backlight sel, J6 indicator bypass, P1 i2c_pin, P2 i2c_pin, SW1 SW_PUSH-MX_W_LED, SW10 SW_PUSH-MX_W_LED, SW11 SW_PUSH-MX_W_LED, SW12 SW_PUSH-MX_W_LED, SW13 SW_PUSH-MX_W_LED, SW14 SW_PUSH-MX_W_LED, SW15 SW_PUSH-MX_W_LED, SW16 SW_PUSH-MX_W_LED, SW17 SW_PUSH-MX_W_LED, SW18 SW_PUSH-MX_W_LED, SW19 SW_PUSH-MX_W_LED, SW2 SW_PUSH-MX_W_LED, SW20 SW_PUSH-MX_W_LED, SW21 SW_PUSH-MX_W_LED, SW22 SW_PUSH-MX_W_LED, SW23 SW_PUSH-MX_W_LED, SW24 SW_PUSH-MX_W_LED, SW25 Rotary_Encoder_Switch, SW26 SW_PUSH-MX_W_LED, SW27 SW_PUSH-MX_W_LED, SW28 SW_PUSH-MX_W_LED, SW29 SW_PUSH-MX_W_LED, SW3 SW_PUSH-MX_W_LED, SW30 SW_PUSH-MX_W_LED, SW4 SW_PUSH-MX_W_LED, SW5 SW_PUSH-MX_W_LED, SW6 SW_PUSH-MX_W_LED, SW7 SW_PUSH-MX_W_LED, SW8 SW_PUSH-MX_W_LED, SW9 SW_PUSH-MX_W_LED, U1 ProMicro

Commit message: unknown changes
Connections:
- net GND: now also D37.2 (VSS); no longer D37.4 (VDD)
- net VCC: now also D37.4 (VDD); no longer D37.2 (VSS)
Changed lines of the file:
@@
 	3700 2200 3750 2200
 Wire Wire Line
-	4550 2400 4400 2400
-Wire Wire Line
 	4000 2500 3850 2500
-Wire Wire Line
-	3850 2500 3850 2550
 Wire Wire Line
 	4400 2500 4550 2500
@@
 $EndComp
 $Comp
-L SofleKeyboard:SW_PUSH-MX_W_LED SW4
-U 1 1 5B722A11
-P 9000 3450
-F 0 "SW4" H 9000 3705 50  0000 C CNN
-F 1 "SW_PUSH-MX_W_LED" H 9000 3614 50  0000 C CNN
-F 2 "Button_Switch_Keyboard:SK6812MINI_and_cherry" H 9000 3450 50  0001 C CNN
-F 3 "" H 9000 3450 50  0000 C CNN
-	1    9000 3450
-	1    0    0    -1
-$EndComp
-$Comp
 L SofleKeyboard-rescue:GND-Lily58-cache-Lily58_Pro-rescue #PWR024
 U 1 1 5FEF0394
@@
 L SofleKeyboard-rescue:GND-Lily58-cache-Lily58_Pro-rescue #PWR023
 U 1 1 5FB348BA
-P 3850 2550
-F 0 "#PWR023" H 3850 2300 50  0001 C CNN
-F 1 "GND" H 3855 2377 50  0000 C CNN
-F 2 "" H 3850 2550 50  0001 C CNN
-F 3 "" H 3850 2550 50  0001 C CNN
-	1    3850 2550
+P 4950 2700
+F 0 "#PWR023" H 4950 2450 50  0001 C CNN
+F 1 "GND" H 4955 2527 50  0000 C CNN
+F 2 "" H 4950 2700 50  0001 C CNN
+F 3 "" H 4950 2700 50  0001 C CNN
+	1    4950 2700
 	1    0    0    -1
 $EndComp
@@
 L SofleKeyboard-rescue:VCC-Lily58-cache-Lily58_Pro-rescue #PWR022
 U 1 1 5FB33FDA
-P 4550 2400
-F 0 "#PWR022" H 4550 2250 50  0001 C CNN
-F 1 "VCC" H 4567 2573 50  0000 C CNN
-F 2 "" H 4550 2400 50  0001 C CNN
-F 3 "" H 4550 2400 50  0001 C CNN
-	1    4550 2400
+P 3650 2750
+F 0 "#PWR022" H 3650 2600 50  0001 C CNN
+F 1 "VCC" H 3667 2923 50  0000 C CNN
+F 2 "" H 3650 2750 50  0001 C CNN
+F 3 "" H 3650 2750 50  0001 C CNN
+	1    3650 2750
 	1    0    0    -1
 $EndComp
@@
 NoConn ~ 7950 2250
 NoConn ~ 6400 1550
+$Comp
+L SofleKeyboard:SW_PUSH-MX_W_LED SW4
+U 1 1 5B722A11
+P 9000 3450
+F 0 "SW4" H 9000 3705 50  0000 C CNN
+F 1 "SW_PUSH-MX_W_LED" H 9000 3614 50  0001 C CNN
+F 2 "Button_Switch_Keyboard:SK6812MINI_and_cherry" H 9000 3450 50  0001 C CNN
+F 3 "" H 9000 3450 50  0000 C CNN
+	1    9000 3450
+	1    0    0    -1
+$EndComp
+Wire Wire Line
+	3650 2750 3850 2750
+Wire Wire Line
+	3850 2500 3850 2750
+Wire Wire Line
+	4400 2400 4950 2400
+Wire Wire Line
+	4950 2400 4950 2700
 $EndSCHEMATC
