File: Case/Sofle_RGB/PCBTop/SofleKeyboardTopPlate.kicad_pcb (KiCad board)
At the start: 2 copper layers, 143.4 x 111.8 mm, 9 parts

Commit message: fixed top and bottom plate hole sizes
Parts:
- moved G*** 9.22 mm to (193.0, 126.2)
- moved G*** 9.22 mm to (192.2, 126.2)
- moved G*** 4.81 mm to (94.5, 117.3)
- moved G*** 4.74 mm to (95.5, 117.3)
Other:
- board text added: "Sofle RGB - Dane Evans"
- board text added: "Sofle RGB v1.1, Dane Evans"
- board text removed: "Sofle RGB v1.0, Dane Evans"
Changed lines of the file:
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@@
   (general
     (thickness 1.6)
-    (drawings 164)
+    (drawings 166)
     (tracks 0)
     (zones 0)
@@
   (layers
     (0 F.Cu signal)
-    (31 B.Cu signal hide)
+    (31 B.Cu signal)
     (32 B.Adhes user hide)
     (33 F.Adhes user hide)
@@
     (mod_text_size 1 1)
     (mod_text_width 0.15)
-    (pad_size 4 4)
+    (pad_size 4.7 4.7)
     (pad_drill 2.2)
     (pad_to_mask_clearance 0.2)
@@
   )
   (module dane:gecko-logo (layer F.Cu)
-    (at 92.545 121.695)
+    (at 94.495 117.3)
     (fp_text reference G*** (at 0 0) (layer F.SilkS) hide
       (effects (font (size 1.524 1.524) (thickness 0.3)))
@@
   )
   (module dane:gecko-logo (layer B.Cu)
-    (at 93.495 121.595 180)
+    (at 95.495 117.3 180)
     (fp_text reference G*** (at 0 0) (layer B.SilkS) hide
       (effects (font (size 1.524 1.524) (thickness 0.3)) (justify mirror))
@@
   )
   (module dane:gecko-logo (layer B.Cu)
-    (at 201.995 124.195 180)
+    (at 192.995 126.195 180)
     (fp_text reference G*** (at 0 0) (layer B.SilkS) hide
       (effects (font (size 1.524 1.524) (thickness 0.3)) (justify mirror))
@@
       (effects (font (size 0.29972 0.29972) (thickness 0.0762)))
     )
-    (pad "" thru_hole circle (at 0 0 180) (size 4.7 4.7) (drill 4.1) (layers *.Cu *.Mask Dwgs.User)
+    (pad "" thru_hole circle (at 0 0 180) (size 4.7 4.7) (drill 2.2) (layers *.Cu *.Mask Dwgs.User)
       (clearance 0.3))
   )
@@
       (effects (font (size 0.29972 0.29972) (thickness 0.0762)))
     )
-    (pad "" thru_hole circle (at -0.025 -0.075 90) (size 4.7 4.7) (drill 4.1) (layers *.Cu *.Mask Dwgs.User)
+    (pad "" thru_hole circle (at -0.025 -0.075 90) (size 4.7 4.7) (drill 2.2) (layers *.Cu *.Mask Dwgs.User)
       (clearance 0.3))
   )
@@
       (effects (font (size 0.29972 0.29972) (thickness 0.0762)))
     )
-    (pad "" thru_hole circle (at -0.175 -0.025 90) (size 4.7 4.7) (drill 4.1) (layers *.Cu *.Mask Dwgs.User)
+    (pad "" thru_hole circle (at -0.175 -0.025 90) (size 4.7 4.7) (drill 2.2) (layers *.Cu *.Mask Dwgs.User)
       (clearance 0.3))
   )
@@
       (effects (font (size 0.29972 0.29972) (thickness 0.0762)))
     )
-    (pad "" thru_hole circle (at 0.025 -0.075 90) (size 4.7 4.7) (drill 4.1) (layers *.Cu *.Mask Dwgs.User)
+    (pad "" thru_hole circle (at 0.025 -0.075 90) (size 4.7 4.7) (drill 2.2) (layers *.Cu *.Mask Dwgs.User)
       (clearance 0.3))
   )
@@
       (effects (font (size 0.29972 0.29972) (thickness 0.0762)))
     )
-    (pad "" thru_hole circle (at -0.225 -0.275 90) (size 4.7 4.7) (drill 4.1) (layers *.Cu *.Mask Dwgs.User)
+    (pad "" thru_hole circle (at -0.225 -0.275 90) (size 4.7 4.7) (drill 2.2) (layers *.Cu *.Mask Dwgs.User)
       (clearance 0.3))
   )
   (module dane:gecko-logo (layer F.Cu)
-    (at 201.245 124.195)
+    (at 192.245 126.195)
     (fp_text reference G*** (at 0 0) (layer F.SilkS) hide
       (effects (font (size 1.524 1.524) (thickness 0.3)))
@@
       (xy 0.54669 -1.86187) (xy 0.574235 -1.866205) (xy 0.601318 -1.845968)) (layer F.Mask) (width 0.01))
   )
+  (gr_text "Sofle RGB - Dane Evans\n" (at 101.495 114.3) (layer B.SilkS)
+    (effects (font (size 1 1) (thickness 0.2)) (justify mirror))
+  )
+  (gr_text "Sofle RGB - Dane Evans\n" (at 100.995 114.3) (layer F.SilkS)
+    (effects (font (size 1 1) (thickness 0.2)))
+  )
   (gr_line (start 112.995 38) (end 113.395 37.9) (layer Edge.Cuts) (width 0.15))
   (gr_line (start 112.695 38.1) (end 112.995 38) (layer Edge.Cuts) (width 0.15))
@@
   (gr_line (start 111.995 96.8) (end 111.995 39.045) (layer Edge.Cuts) (width 0.15))
   (gr_line (start 90.3 97.8) (end 110.995 97.8) (layer Edge.Cuts) (width 0.15))
-  (gr_text "Sofle RGB v1.0, Dane Evans" (at 202.245 128.695 21) (layer F.Cu)
+  (gr_text "Sofle RGB v1.1, Dane Evans" (at 202.245 128.695 21) (layer F.Cu)
     (effects (font (size 1 1) (thickness 0.2)))
   )
-  (gr_text "Sofle RGB v1.0, Dane Evans" (at 201.995 128.695 21) (layer B.Cu)
+  (gr_text "Sofle RGB v1.1, Dane Evans" (at 201.995 128.695 21) (layer B.Cu)
     (effects (font (size 1 1) (thickness 0.2)) (justify mirror))
   )
-  (gr_text "Original Sofle design by Josef Adamacik" (at 130.895 79.1 90) (layer F.SilkS)
+  (gr_text "Original Sofle design by Josef Adamacik" (at 130.895 79.1 90) (layer F.Cu)
     (effects (font (size 1 1) (thickness 0.2)))
   )
-  (gr_text "Original Sofle design by Josef Adamacik" (at 130.995 79.3 270) (layer B.SilkS)
+  (gr_text "Original Sofle design by Josef Adamacik" (at 130.995 79.3 270) (layer B.Cu)
     (effects (font (size 1 1) (thickness 0.2)) (justify mirror))
   )
-  (gr_text https://josefadamcik.github.io/SofleKeyboard/ (at 150.095 80.5 90) (layer F.SilkS)
+  (gr_text https://josefadamcik.github.io/SofleKeyboard/ (at 150.095 80.5 90) (layer F.Cu)
     (effects (font (size 1 1) (thickness 0.15)))
   )
-  (gr_text https://josefadamcik.github.io/SofleKeyboard/ (at 150.395 80.5 270) (layer B.SilkS)
+  (gr_text https://josefadamcik.github.io/SofleKeyboard/ (at 150.395 80.5 270) (layer B.Cu)
     (effects (font (size 1 1) (thickness 0.15)) (justify mirror))
   )
@@
   (gr_line (start 93.545 147.645) (end 83.295 129.845) (layer Edge.Cuts) (width 0.1))
   (gr_line (start 226.278881 45.442807) (end 226.365281 45.623672) (layer Edge.Cuts) (width 0.1))
-  (zone (net 0) (net_name "") (layer B.Cu) (hatch edge 0.508)
-    (connect_pads (clearance 0.508))
-    (min_thickness 0.254)
-    (fill yes (arc_segments 32) (thermal_gap 0.508) (thermal_bridge_width 0.508))
-    (polygon
-      (pts
-        (xy -13.208 20.32) (xy -10.922 99.822) (xy -31.75 103.124) (xy -41.148 117.094) (xy -64.516 118.364)
-        (xy -80.01 113.284) (xy -98.806 111.76) (xy -137.922 127.508) (xy -152.908 94.996) (xy -153.924 72.898)
-        (xy -130.556 72.898) (xy -130.556 15.748) (xy -51.816 13.97)
-      )
-    )
-  )
   (zone (net 0) (net_name "") (layer F.Cu) (hatch edge 0.508)
     (connect_pads (clearance 0.508))
